File: CAD/JiggleBilly/Lib/JiggleBilly_SAO_V1/JiggleBilly.kicad_pcb (KiCad board)
At the start: 2 copper layers, 86.3 x 94.7 mm, 10 parts, among them X1 Badgelife_sao_connector_v169b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

Commit message: Changes from sending PCBs for Estimate
Other:
- rule pad_to_mask_clearance: 0.2 -> 0
Changed lines of the file:
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@@
 			(dielectric_constraints no)
 		)
-		(pad_to_mask_clearance 0.2)
-		(allow_soldermask_bridges_in_footprints no)
+		(pad_to_mask_clearance 0)
+		(allow_soldermask_bridges_in_footprints yes)
 		(pcbplotparams
-			(layerselection 0x00010f0_80000001)
+			(layerselection 0x00010fc_ffffffff)
 			(plot_on_all_layers_selection 0x0000000_00000000)
 			(disableapertmacros no)
-			(usegerberextensions no)
-			(usegerberattributes yes)
-			(usegerberadvancedattributes yes)
-			(creategerberjobfile yes)
+			(usegerberextensions yes)
+			(usegerberattributes no)
+			(usegerberadvancedattributes no)
+			(creategerberjobfile no)
 			(dashed_line_dash_ratio 12.000000)
 			(dashed_line_gap_ratio 3.000000)
@@
 			(psa4output no)
 			(plotreference yes)
-			(plotvalue yes)
+			(plotvalue no)
 			(plotfptext yes)
 			(plotinvisibletext no)
 			(sketchpadsonfab no)
-			(subtractmaskfromsilk no)
+			(subtractmaskfromsilk yes)
 			(outputformat 1)
 			(mirror no)
-			(drillshape 1)
+			(drillshape 0)
 			(scaleselection 1)
-			(outputdirectory "gerbers/")
+			(outputdirectory "../../../../Outputs/Gerber and Drill/JLCPCB/")
 		)
 	)
